Commit message: Scanner in right position and orientation

File: assets/scenes/bunker_with_arm/bunker_with_arm.urdf.xacro (robot description, xacro)
@@ -61,4 +61,4 @@
     <child link="camera_link"/> <!-- Direct reference to Orbbec's link -->
   </joint>
-  <xacro:include filename="${orbbec_path}/urdf/gemini_335_336.urdf.xacro" />
+  <xacro:include filename="${orbbec_path}/urdf/my_orbbec.urdf" />
 </robot>

File: assets/sensors/keyence_experimental/urdf/lj_v7200_macro.xacro (robot description, xacro)
@@ -29,5 +29,13 @@
       <parent link="${prefix}lj_v7200_optical_frame"/>
       <child  link="${prefix}lj_v7200_frame"/>
-   </joint>
+    </joint>
+    <!-- Connect the virtual root to the actual base link
+    <link name="base_link"/>
+    <joint name="base_link_to_lj_v7200_optical_frame" type="fixed">
+      <parent link="base_link"/>
+      <child link="${prefix}lj_v7200_optical_frame"/>
+      <origin rpy="0 0 0" xyz="0.0 0.0 0.0"/>
+    </joint>
+  <xacro:lj_v7200 prefix=""/>-->
   </xacro:macro>
 </robot>
