Commit message: Torch tip added to .xacro of scene

File: assets/scenes/my_arm.urdf.xacro (robot description, xacro)
@@ -26,4 +26,11 @@
     <child link="torch"/>
   </joint>
+  <!-- ===== WELDING TORCH TIP ===== -->
+  <link name="torch_tip" />
+  <joint name="wrist_3_link_torch_tip_fixed_joint" type="fixed">
+    <origin xyz="0.0 -0.106 0.367" rpy="0 -0.018 -0.004"/> <!-- Good as on 21 August 2025 -->
+    <parent link="wrist_3_link"/>
+    <child link="torch_tip"/>
+  </joint>
   <!-- ===== KEYENCE LASER SCANNER ===== -->
   <joint name="wrist_3_link_lj_v7200_frame" type="fixed">
