Commit message: "file://..." in ur10_nominal.urdf replaced by "package://..."

File: assets/robots/ur_description/urdf/ur10_nominal.urdf (robot description, URDF)
Before this commit: robot ur10, 13 links, 11 joints
Links:
- link base_link_inertia: geometry collision mesh filename=package://robots/ur_description/meshes/ur10/collision/base.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; visual mesh filename=package://robots/ur_description/meshes/ur10/visual/base.dae
- link forearm_link: geometry collision mesh filename=package://robots/ur_description/meshes/ur10/collision/forea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; visual mesh filename=package://robots/ur_description/meshes/ur10/visual/forearm.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
- link shoulder_link: geometry collision mesh filename=package://robots/ur_description/meshes/ur10/collision/shoul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; visual mesh filename=package://robots/ur_description/meshes/ur10/visual/shoulder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
- link upper_arm_link: geometry collision mesh filename=package://robots/ur_description/meshes/ur10/collision/upper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; visual mesh filename=package://robots/ur_description/meshes/ur10/visual/upperarm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
- link wrist_1_link: geometry collision mesh filename=package://robots/ur_description/meshes/ur10/collision/wrist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; visual mesh filename=package://robots/ur_description/meshes/ur10/visual/wrist1.d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
- link wrist_2_link: geometry collision mesh filename=package://robots/ur_description/meshes/ur10/collision/wrist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; visual mesh filename=package://robots/ur_description/meshes/ur10/visual/wrist2.d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
- link wrist_3_link: geometry collision mesh filename=package://robots/ur_description/meshes/ur10/collision/wrist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; visual mesh filename=package://robots/ur_description/meshes/ur10/visual/wrist3.d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
